File: pcb/quantar-interface/quantar-interface.sch (KiCad schematic (older format))
At the start: 71 parts

Commit message: Done with schematic, ready to route
Parts:
- removed C? (x2): 4.7uF, symbol Device:CP
- removed T? (x2): 600 Ohm 1:1, symbol Device:Transformer_1P_1S
- added C13, C8: 4.7uF, Capacitor_SMD:CP_Elec_4x5.4, symbol Device:C
- added C29, C33: 1uF, Capacitor_SMD:CP_Elec_4x4.5, symbol Device:CP
- added C3, C4: 47p, Capacitor_SMD:C_0805_2012Metric_Pad1.15x1.40mm_HandSolder, symbol Device:C
- added C30: 10uF, Capacitor_SMD:CP_Elec_4x5.8, symbol Device:CP
- added C31: 0.01uF, Capacitor_SMD:C_0805_2012Metric_Pad1.15x1.40mm_HandSolder, symbol Device:C
- added C32, C35, C36: 0.1uF, Capacitor_SMD:C_0805_2012Metric_Pad1.15x1.40mm_HandSolder, symbol Device:C
- added C34: 47pF, Capacitor_SMD:C_0805_2012Metric_Pad1.15x1.40mm_HandSolder, symbol Device:C
- added D11: LED_HEARTBEAT, LED_SMD:LED_0805_2012Metric_Pad1.15x1.40mm_HandSolder, symbol Device:LED
- added D12, D14: 1N4148, Diode_SMD:D_SOD-523, symbol Device:D
- added D13: LED_ALARM, LED_SMD:LED_0805_2012Metric_Pad1.15x1.40mm_HandSolder, symbol Device:LED
- added D15: LED_SPARE_OUT, LED_SMD:LED_0805_2012Metric_Pad1.15x1.40mm_HandSolder, symbol Device:LED
- added D16: LED_PTT, LED_SMD:LED_0805_2012Metric_Pad1.15x1.40mm_HandSolder, symbol Device:LED
- added D17: LED_WDOG, LED_SMD:LED_0805_2012Metric_Pad1.15x1.40mm_HandSolder, symbol Device:LED
- added D18: LED_PL, LED_SMD:LED_0805_2012Metric_Pad1.15x1.40mm_HandSolder, symbol Device:LED
- added D19: LED_COS, LED_SMD:LED_0805_2012Metric_Pad1.15x1.40mm_HandSolder, symbol Device:LED
- added D20: LED_FS, LED_SMD:LED_0805_2012Metric_Pad1.15x1.40mm_HandSolder, symbol Device:LED
- added D21: LED_TI, LED_SMD:LED_0805_2012Metric_Pad1.15x1.40mm_HandSolder, symbol Device:LED
- added D22: LED_SD, LED_SMD:LED_0805_2012Metric_Pad1.15x1.40mm_HandSolder, symbol Device:LED
- added D23: LED_SI, LED_SMD:LED_0805_2012Metric_Pad1.15x1.40mm_HandSolder, symbol Device:LED
- added H1, H2, H3, H4: MountingHole, MountingHole:MountingHole_4mm, symbol Mechanical:MountingHole
- added J4: GPIO, Connector_PinHeader_2.54mm:PinHeader_1x03_P2.54mm_Vertical, symbol Connector_Generic:Conn_01x03
- added J6: Ext. Alarm Contact, Connector_Phoenix_MC:PhoenixContact_MC_1,5_3-G-3.5_1x03_P3.50mm_Horizontal, symbol Connector:Screw_Terminal_01x03
- added J7: Ext. TX Inhb., Connector_Phoenix_MC:PhoenixContact_MC_1,5_2-G-3.5_1x02_P3.50mm_Horizontal, symbol Connector:Screw_Terminal_01x02
- added J8: Quantar, Connector_Phoenix_MC:PhoenixContact_MC_1,5_13-G-3.5_1x13_P3.50mm_Horizontal, symbol Connector:Screw_Terminal_01x13
- added JP1: MSEL, Jumper:SolderJumper-3_P1.3mm_Bridged12_RoundedPad1.0x1.5mm_NumberLabels, symbol Jumper:SolderJumper_3_Open
- added JP2: Watchdog Bypass, Connector_PinHeader_2.54mm:PinHeader_1x03_P2.54mm_Vertical, symbol Jumper:Jumper_3_Bridged12
- added K1: G6S-2, Relay_THT:Relay_DPDT_Omron_G6S-2, symbol Relay:G6S-2
- added Q2, Q3, Q4, Q5, Q6: 2N7002, Package_TO_SOT_SMD:SOT-23, symbol Transistor_FET:2N7002
- added R12, R20: 1M, Resistor_SMD:R_0805_2012Metric_Pad1.15x1.40mm_HandSolder, symbol Device:R
- added R17, R23, R24, R25, R26, R27, R28, R29, R30, R31, R32, R33, R38, R39, R41, R42, R43, R44: 330, Resistor_SMD:R_0805_2012Metric_Pad1.15x1.40mm_HandSolder, symbol Device:R
- added R18, R19, R21: 4.7K, Resistor_SMD:R_0805_2012Metric_Pad1.15x1.40mm_HandSolder, symbol Device:R
- added R2, R3, R45: 22, Resistor_SMD:R_0805_2012Metric_Pad1.15x1.40mm_HandSolder, symbol Device:R
- added R22: 2.2K, Resistor_SMD:R_0805_2012Metric_Pad1.15x1.40mm_HandSolder, symbol Device:R
- added R34, R35, R36, R37, R46: 10K, Resistor_SMD:R_0805_2012Metric_Pad1.15x1.40mm_HandSolder, symbol Device:R
- added R40: 0, Resistor_SMD:R_0805_2012Metric_Pad1.15x1.40mm_HandSolder, symbol Device:R
- added SW1: SW_TX_INHB, Button_Switch_THT:SW_Slide_1P2T_CK_OS102011MS2Q, symbol Switch:SW_SPDT
- added SW2: SW_PTT_INHB, Button_Switch_THT:SW_Slide_1P2T_CK_OS102011MS2Q, symbol Switch:SW_SPDT
- added T1, T2: Transformer, quantar-interface:Transformer, symbol quantar-interface:Transformer
- added TP1: EEPROM CS, TestPoint:TestPoint_Pad_1.0x1.0mm, symbol Connector:TestPoint
- added TP10: Prereg, TestPoint:TestPoint_Pad_1.0x1.0mm, symbol Connector:TestPoint
- added TP11: 5V Analog, TestPoint:TestPoint_Pad_1.0x1.0mm, symbol Connector:TestPoint
- added TP12: TP HB, TestPoint:TestPoint_Pad_1.0x1.0mm, symbol Connector:TestPoint
- added TP13: TP HB Pulse, TestPoint:TestPoint_Pad_1.0x1.0mm, symbol Connector:TestPoint
- added TP14: TP ALARM, TestPoint:TestPoint_Pad_1.0x1.0mm, symbol Connector:TestPoint
- added TP15: TP SPARE OUTP, TestPoint:TestPoint_Pad_1.0x1.0mm, symbol Connector:TestPoint
- added TP16: TP PL, TestPoint:TestPoint_Pad_1.0x1.0mm, symbol Connector:TestPoint
- added TP17: TP PTT, TestPoint:TestPoint_Pad_1.0x1.0mm, symbol Connector:TestPoint
- added TP18: TP WDOG, TestPoint:TestPoint_Pad_1.0x1.0mm, symbol Connector:TestPoint
- added TP19: TP COS, TestPoint:TestPoint_Pad_1.0x1.0mm, symbol Connector:TestPoint
- added TP2: EEPROM SK, TestPoint:TestPoint_Pad_1.0x1.0mm, symbol Connector:TestPoint
- added TP20: TP TX INHB, TestPoint:TestPoint_Pad_1.0x1.0mm, symbol Connector:TestPoint
- added TP21: TP SCAN DISBL, TestPoint:TestPoint_Pad_1.0x1.0mm, symbol Connector:TestPoint
- added TP22: TP SPARE INP, TestPoint:TestPoint_Pad_1.0x1.0mm, symbol Connector:TestPoint
- added TP23: TP SCAN DISBL ISO, TestPoint:TestPoint_Pad_1.0x1.0mm, symbol Connector:TestPoint
- added TP24: TP SPARE INP ISO, TestPoint:TestPoint_Pad_1.0x1.0mm, symbol Connector:TestPoint
- added TP25: TP WDOG ISO, TestPoint:TestPoint_Pad_1.0x1.0mm, symbol Connector:TestPoint
- added TP26: TP TX INHB ISO, TestPoint:TestPoint_Pad_1.0x1.0mm, symbol Connector:TestPoint
- added TP27: TP PTT Disable, TestPoint:TestPoint_Pad_1.0x1.0mm, symbol Connector:TestPoint
- added TP28: LOR, TestPoint:TestPoint_Pad_1.0x1.0mm, symbol Connector:TestPoint
- added TP3: EEPROM DR, TestPoint:TestPoint_Pad_1.0x1.0mm, symbol Connector:TestPoint
- added TP4: EEPROM DW, TestPoint:TestPoint_Pad_1.0x1.0mm, symbol Connector:TestPoint
- added TP5: Mic In, TestPoint:TestPoint_Pad_1.0x1.0mm, symbol Connector:TestPoint
- added TP6: 12V, TestPoint:TestPoint_Pad_1.0x1.0mm, symbol Connector:TestPoint
- added TP7: Amp Out, TestPoint:TestPoint_Pad_1.0x1.0mm, symbol Connector:TestPoint
- added TP8: RX In, TestPoint:TestPoint_Pad_1.0x1.0mm, symbol Connector:TestPoint
- added TP9: 5V Digital, TestPoint:TestPoint_Pad_1.0x1.0mm, symbol Connector:TestPoint
- added U10, U11, U12, U13, U14, U8, U9: 4N27, Package_DIP:DIP-6_W7.62mm_LongPads, symbol Isolator:4N27
- added U15: 74HC14, Package_SO:SO-8_3.9x4.9mm_P1.27mm, symbol 74xx:74HC14
- added U7: LM555, Package_SO:SOIC-8_3.9x4.9mm_P1.27mm, symbol Timer:LM555
- C1, C18, C7: renamed from C?; footprint (none) -> Capacitor_SMD:CP_Elec_4x5.4
- C10, C14, C15, C2, C6: renamed from C?; footprint (none) -> Capacitor_SMD:C_0805_2012Metric_Pad1.15x1.40mm_HandSolder
- C11, C12, C16, C19, C23, C5, C9: renamed from C?; footprint (none) -> Capacitor_SMD:CP_Elec_6.3x5.4
- C17, C24, C27: renamed from C?; footprint (none) -> Capacitor_SMD:C_1206_3216Metric_Pad1.42x1.75mm_HandSolder
- C20, C25, C26, C28: renamed from C?; footprint (none) -> Capacitor_SMD:CP_Elec_4x5.8
- C21, C22: renamed from C?; value C -> 12pF; footprint (none) -> Capacitor_SMD:C_0805_2012Metric_Pad1.15x1.40mm_HandSolder
- D1, D10, D8, D9: renamed from D?; footprint (none) -> LED_SMD:LED_0805_2012Metric_Pad1.15x1.40mm_HandSolder
- D2, D3: renamed from D?; value D_Schottky -> B340LA; footprint (none) -> Diode_SMD:D_SMA_Handsoldering
- D4, D5, D6, D7: renamed from D?; footprint (none) -> Diode_SMD:D_SOD-323_HandSoldering
- F1, F2: renamed from F?; footprint (none) -> Fuse:Fuse_2920_7451Metric_Pad2.10x5.45mm_HandSolder
- FB1, FB2: renamed from FB?; footprint (none) -> Inductor_SMD:L_0603_1608Metric_Pad1.05x0.95mm_HandSolder
- J1: renamed from J?; footprint (none) -> Connector_BarrelJack:BarrelJack_Horizontal
- J2: renamed from J?; footprint (none) -> Connector_USB:USB_A_Stewart_SS-52100-001_Horizontal
- J3: renamed from J?; footprint (none) -> Connector_USB:USB_B_OST_USB-B1HSxx_Horizontal
- J5: renamed from J?; footprint (none) -> Connector_Phoenix_MC:PhoenixContact_MC_1,5_5-G-3.5_1x05_P3.50mm_Horizontal
- L1: renamed from L?; footprint (none) -> Inductor_SMD:L_12x12mm_H4.5mm
- L2: renamed from L?; footprint (none) -> Inductor_SMD:L_1008_2520Metric
- Q1: renamed from Q?; footprint (none) -> Package_TO_SOT_SMD:SOT-23
- R1, R10, R11, R13, R14, R15, R16, R4, R5, R6, R7, R8, R9: renamed from R?; footprint (none) -> Resistor_SMD:R_0805_2012Metric_Pad1.15x1.40mm_HandSolder
- RV1, RV2: renamed from RV?; footprint (none) -> Potentiometer_THT:Potentiometer_Bourns_3296W_Vertical
- U1, U2: renamed from U?; footprint (none) -> Package_SO:SO-8_3.9x4.9mm_P1.27mm
- U4: renamed from U?; footprint (none) -> Package_TO_SOT_SMD:TO-263-5_TabPin6
- U5: renamed from U?; footprint (none) -> Package_QFP:LQFP-48_7x7mm_P0.5mm
- U6: renamed from U?; footprint (none) -> Package_TO_SOT_SMD:SOT-223-3_TabPin2
- Y1: renamed from Y?; footprint (none) -> Crystal:Crystal_SMD_HC49-SD
- gave numbers to parts that had none: 1
Connections:
- net labels added: ALARM, COS, GPIO7, GPIO8, HEARTBEAT, PL, PTT, SCAN_DISABLE, SPARE_INPUT, SPARE_OUTPUT, STATION_5V, STATION_ALARM, STATION_COS_RELAY_A, STATION_COS_RELAY_B, STATION_FAILSOFT, STATION_GND, STATION_PL_ACTIVE, STATION_PTT_LED+, STATION_PTT_LED-, STATION_SCAN_DISABLE, STATION_SPARE_INPUT, STATION_SPARE_OUTPUT, STATION_TX_INHIBIT, TX_INHB, WATCHDOG_OK
- wire segments 268 -> 580
- no-connect marks 13 -> 27
Other:
- note added: "3.3V Levels - pulled up in CM119A\nH - No PL (normal)\nL - Station TXing PL"
- note added: "3.3V Levels - pulled up in CM119A\nH - Not receiving (normal)\nL - Receiving"
- note added: "3.3V Levels - pullup in CM119A"
- note added: "3.3V Levels - pullup in CM119A\nH - Alarm\nL - No Alarm (normal)"
- note added: "3.3V Levels\nH - Block all transmissions\nL - Enable transmitter (Normal)"
- note added: "3.3V Levels\nH - Key up station\nL - Dekey station (normal)"
- note added: "3.3V Levels\nH - Stop scanning\nL - Scan (Normal)"
- note added: "Alarm"
- note added: "Alarm Output"
- note added: "Audio I/O"
- note added: "Carrier-operated Squelch"
- note added: "Lit LED indicates\nPC conn. good"
- note added: "Note: Indicated Quantar pin numbers\nand functions are specific to W1XM’s\nunit and require proper configuration\nin the WildCard tables."
- note added: "Note: Spare Input\nand Output are from\nthe Quantar’s perspective."
- note added: "Note: This pinout does not correspond\nto any particular port on the Quantar. User\nmust map these signals to the 50-Pin Telco\nconnector and set up I/O in Wildcard settings."
- note added: "PL Active"
- note added: "PTT and Failsoft"
- note added: "Quantar open-collector\noutput (pin 36, Aux Out 1)\n\nActive (pulled down): Sending PL\nInactive: Not sending PL"
- note added: "Quantar open-collector\noutput (pin 38, Aux Out 3)\n\nActive (pulled down): No Alarm\nInactive: Alarm present"
- note added: "Quantar open-collector\noutput (pin 39, Aux Out 4)"
- note added: "Quantar opto-isolated\ninput. (Pin 22 anode,\n47 cathode, Aux In 9)\n\nActive (Lit): Key up station\nInactive: Dekey station"
- note added: "Quantar transistor\ninput. (Pin 11, Aux In 1)\n\nLo / Hi-Z: TX Allowed\nHi: TX Inhibited"
- note added: "Quantar transistor\ninput. (Pin 12, Aux In 2)\n\nLo / Hi-Z: Failsoft\nHi: External controller"
- note added: "Quantar transistor\ninput. (Pin 13, Aux In 3)\n\nLo / Hi-Z: Scan other CH\nHi: Do not scan"
- note added: "Quantar transistor\ninput. (Pin 14, Aux In 4)"
- note added: "Require watchdog to be\nOK (H) to key up station"
- note added: "Scan Disable"
- note added: "Signal is high (5V)\nwhen PC comms\nare good."
- note added: "Spare Input"
- note added: "Spare Output"
- note added: "TX Inhibit"
- note added: "Testing Only\nDNP"
- note added: "To N.O. relay contact\ninside Quantar cabinet\n(Quantar pins 18, 43, Aux Out 7)\n\nClosed: Receiving\nOpen: Not receiving"
- note added: "USB Codec"
- note added: "USB Power Out to RPi"
- note added: "Unused"
- note added: "Watchdog"
- note removed: "TODO:\n 1) Add test points\n 2) Revisit decouplng caps"
- note removed: "USB Power Out"
- moved on the sheet: C1, C10, C11, C12, C14, C15, C16, C17, C18, C19, C2, C20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

Commit message: Correct package for 74HC14; Number the pad for the AP1506
Parts:
- U15: footprint Package_SO:SO-8_3.9x4.9mm_P1.27mm -> Package_SO:SOIC-14_3.9x8.7mm_P1.27mm
Changed lines of the file:
@@
 F 0 "U15" H 17950 6717 50  0000 C CNN
 F 1 "74HC14" H 17950 6626 50  0000 C CNN
-F 2 "Package_SO:SO-8_3.9x4.9mm_P1.27mm" H 17950 6400 50  0001 C CNN
+F 2 "Package_SO:SOIC-14_3.9x8.7mm_P1.27mm" H 17950 6400 50  0001 C CNN
 F 3 "http://www.ti.com/lit/gpn/sn74HC14" H 17950 6400 50  0001 C CNN
 	1    17950 6400
@@
 F 0 "U15" H 21880 4096 50  0000 L CNN
 F 1 "74HC14" H 21880 4005 50  0000 L CNN
-F 2 "Package_SO:SO-8_3.9x4.9mm_P1.27mm" H 21650 4050 50  0001 C CNN
+F 2 "Package_SO:SOIC-14_3.9x8.7mm_P1.27mm" H 21650 4050 50  0001 C CNN
 F 3 "http://www.ti.com/lit/gpn/sn74HC14" H 21650 4050 50  0001 C CNN
 	7    21650 4050
@@
 F 0 "U15" H 17950 8367 50  0000 C CNN
 F 1 "74HC14" H 17950 8276 50  0000 C CNN
-F 2 "Package_SO:SO-8_3.9x4.9mm_P1.27mm" H 17950 8050 50  0001 C CNN
+F 2 "Package_SO:SOIC-14_3.9x8.7mm_P1.27mm" H 17950 8050 50  0001 C CNN
 F 3 "http://www.ti.com/lit/gpn/sn74HC14" H 17950 8050 50  0001 C CNN
 	3    17950 8050
@@
 F 0 "U15" H 17950 10717 50  0000 C CNN
 F 1 "74HC14" H 17950 10626 50  0000 C CNN
-F 2 "Package_SO:SO-8_3.9x4.9mm_P1.27mm" H 17950 10400 50  0001 C CNN
+F 2 "Package_SO:SOIC-14_3.9x8.7mm_P1.27mm" H 17950 10400 50  0001 C CNN
 F 3 "http://www.ti.com/lit/gpn/sn74HC14" H 17950 10400 50  0001 C CNN
 	4    17950 10400
@@
 F 0 "U15" H 17950 12567 50  0000 C CNN
 F 1 "74HC14" H 17950 12476 50  0000 C CNN
-F 2 "Package_SO:SO-8_3.9x4.9mm_P1.27mm" H 17950 12250 50  0001 C CNN
+F 2 "Package_SO:SOIC-14_3.9x8.7mm_P1.27mm" H 17950 12250 50  0001 C CNN
 F 3 "http://www.ti.com/lit/gpn/sn74HC14" H 17950 12250 50  0001 C CNN
 	5    17950 12250
@@
 F 0 "U15" H 21900 6417 50  0000 C CNN
 F 1 "74HC14" H 21900 6326 50  0000 C CNN
-F 2 "Package_SO:SO-8_3.9x4.9mm_P1.27mm" H 21900 6100 50  0001 C CNN
+F 2 "Package_SO:SOIC-14_3.9x8.7mm_P1.27mm" H 21900 6100 50  0001 C CNN
 F 3 "http://www.ti.com/lit/gpn/sn74HC14" H 21900 6100 50  0001 C CNN
 	6    21900 6100

Commit message: Schematic revisions, first draft of layout
Parts:
- removed C30: 10uF, Capacitor_SMD:CP_Elec_4x5.8, symbol Device:CP
- removed TP12: TP HB, TestPoint:TestPoint_Pad_1.0x1.0mm, symbol Connector:TestPoint
- removed TP13: TP HB Pulse, TestPoint:TestPoint_Pad_1.0x1.0mm, symbol Connector:TestPoint
- removed TP23: TP SCAN DISBL ISO, TestPoint:TestPoint_Pad_1.0x1.0mm, symbol Connector:TestPoint
- removed TP24: TP SPARE INP ISO, TestPoint:TestPoint_Pad_1.0x1.0mm, symbol Connector:TestPoint
- removed TP25: TP WDOG ISO, TestPoint:TestPoint_Pad_1.0x1.0mm, symbol Connector:TestPoint
- removed TP26: TP TX INHB ISO, TestPoint:TestPoint_Pad_1.0x1.0mm, symbol Connector:TestPoint
- added F3, F4: PTC 1A, Fuse:Fuse_1210_3225Metric_Pad1.42x2.65mm_HandSolder, symbol Device:Polyfuse_Small
- added FB3: Ferrite, Inductor_SMD:L_0805_2012Metric_Pad1.15x1.40mm_HandSolder, symbol Device:Ferrite_Bead_Small
- added J9: 5V Out, Connector_PinHeader_2.54mm:PinHeader_1x02_P2.54mm_Vertical, symbol Connector_Generic:Conn_01x02
- added unit 2 of U15
- C13, C8: footprint Capacitor_SMD:CP_Elec_4x5.4 -> Capacitor_SMD:C_0805_2012Metric_Pad1.15x1.40mm_HandSolder
- FB1, FB2: footprint Inductor_SMD:L_0603_1608Metric_Pad1.05x0.95mm_HandSolder -> Inductor_SMD:L_0805_2012Metric_Pad1.15x1.40mm_HandSolder
- U10, U11, U12, U13, U14, U8, U9: footprint Package_DIP:DIP-6_W7.62mm_LongPads -> Package_DIP:DIP-6_W7.62mm_SMDSocket_SmallPads
Connections:
- net +5V: now also R20.1, R21.2, U7.4 (R), F4.2
- net GND: now also J9.2 (Pin_2)
- net GNDA: now also T1.1, T2.1; no longer T1.3, T2.3
- net RX_AUDIO_IN: now also T2.3; no longer T2.1
- net RX_AUDIO_LINE2+: now also T2.6; no longer T2.4
- net RX_AUDIO_LINE2-: now also T2.4; no longer T2.6
- net STATION_5V: now also F3.2; no longer J8.1 (Pin_1)
- net STATION_GND: now also U15.3
- net TX_AUDIO_LINE1+: now also T1.6; no longer T1.4
- net TX_AUDIO_LINE1-: now also T1.4; no longer T1.6
- net TX_AUDIO_OUT: now also T1.3; no longer T1.1
- net at C33.1, D12.2 (A), U7.6 (THR)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: now also R20.2; no longer R20.1
- new net: F3.1, FB3.2
- new net: F4.1, J9.1 (Pin_1)
- new net: FB3.1, J8.1 (Pin_1)
- no-connect marks 27 -> 28
Other:
- moved on the sheet: R20, R21

Commit message: Merge split ground planes, connect mounting holes to GND
Parts:
- removed H1, H2, H3, H4: MountingHole, MountingHole:MountingHole_4mm, symbol Mechanical:MountingHole
- removed R15: 0, Resistor_SMD:R_0805_2012Metric_Pad1.15x1.40mm_HandSolder, symbol Device:R
- added H1, H2, H3, H4: MountingHole_Pad, MountingHole:MountingHole_4mm_Pad_Via, symbol Mechanical:MountingHole_Pad
Connections:
- net GND: now also C15.2, C17.2, C20.2, C24.2, C25.2, C26.2, D10.1 (K), R12.2, R5.2, RV1.3, RV2.3, T1.1, T2.1, U2.2 (-), U2.4 (GND), U5.24 (AVSS1), U5.33 (AVSS2), H1.1, H2.1, H3.1, H4.1
- removed net GNDA: C15.2, C17.2, C20.2, C24.2, C25.2, C26.2, C5.2, C7.2, D10.1 (K), R12.2, R5.2, RV1.3, RV2.3, T1.1, T2.1, U2.2 (-), U2.4 (GND), U5.24 (AVSS1), U5.33 (AVSS2)

Commit message: Add BOM
Other:
- note added: "Quantar open-collector\noutput (pin 37, Aux Out 2)"
- note removed: "Quantar open-collector\noutput (pin 39, Aux Out 4)"
Changed lines of the file:
@@
 	13350 14600 17000 14600
 Text Notes 17350 15450 0    50   ~ 0
-Quantar open-collector\noutput (pin 39, Aux Out 4)
+Quantar open-collector\noutput (pin 37, Aux Out 2)
 Entry Wire Line
 	20850 1400 20750 1500

Commit message: Revision B
Parts:
- added R15: 100K, Resistor_SMD:R_0805_2012Metric_Pad1.15x1.40mm_HandSolder, symbol Device:R
- added SW3: Force PTT, Button_Switch_SMD:SW_Push_1P1T_NO_CK_KMR2, symbol Switch:SW_Push
Connections:
- net +5V: now also R32.1
- net GND: now also C5.2, C7.2, R15.1, SW3.2; no longer R32.1, SW2.3 (C)
- net PTT: no longer D16.2 (A)
- net STATION_PTT_LED-: now also D16.1 (K), SW3.1
- net at Q5.1 (G), SW2.2 (B): now also R15.2
- net at R32.2: now also D16.2 (A); no longer D16.1 (K)
- no-connect marks 28 -> 29
Other:
- note added: "Testing\nOnly\nDNP"
- note removed: "Testing Only\nDNP"
- moved on the sheet: D16, Q5, Q6, R32, R40, SW2, TP17, TP18, TP27
